File: pcb/kicad/42.kicad_pcb (KiCad board)
At the start: 2 copper layers, 326.8 x 113.5 mm, 100 parts, among them J1 USB_C_Receptacle, J2 USB_C_Receptacle, J3 USB_C_Receptacle, K1 KEYSW, K10 KEYSW, K11 KEYSW, K12 KEYSW, K13 KEYSW, K14 KEYSW, K15 KEYSW, K16 KEYSW, K17 KEYSW, K18 KEYSW, K19 KEYSW, K2 KEYSW, K20 KEYSW, K21 KEYSW, K22 KEYSW, K23 KEYSW, K24 KEYSW, K25 KEYSW, K26 KEYSW, K27 KEYSW, K28 KEYSW, K29 KEYSW, K3 KEYSW, K30 KEYSW, K31 KEYSW, K32 KEYSW, K33 KEYSW, K34 KEYSW, K35 KEYSW, K36 KEYSW, K37 KEYSW, K38 KEYSW, K39 KEYSW, K4 KEYSW, K40 KEYSW, K41 KEYSW, K42 KEYSW, K5 KEYSW, K6 KEYSW, K7 KEYSW, K8 KEYSW, K9 KEYSW, U1 TEENSY2.0

Commit message: rounded corners, ignore backup saves
Routing:
- net /GND: track 23.5 -> 16.4 mm
- net /+5v: track 16.9 -> 24.0 mm
Changed lines of the file:
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@@
   (general
     (links 355)
-    (no_connects 21)
+    (no_connects 19)
     (area 12.199999 11.949999 339.050001 125.550001)
     (thickness 1.6)
@@
       (net 97 /+5v))
   )
+  (gr_arc (start 17 88.5) (end 17 93.25) (angle 90) (layer Edge.Cuts) (width 0.1))
+  (gr_arc (start 17.25 24.75) (end 12.25 24.75) (angle 90) (layer Edge.Cuts) (width 0.1))
+  (gr_arc (start 334 24.75) (end 334 19.75) (angle 90) (layer Edge.Cuts) (width 0.1))
+  (gr_arc (start 334.25 88.5) (end 339 88.5) (angle 90) (layer Edge.Cuts) (width 0.1))
+  (gr_arc (start 185.25 120.5) (end 185.25 125.5) (angle 90) (layer Edge.Cuts) (width 0.1))
+  (gr_arc (start 166 120.5) (end 171 120.5) (angle 90) (layer Edge.Cuts) (width 0.1))
+  (gr_arc (start 185.25 22.25) (end 180.25 22.25) (angle 90) (layer Edge.Cuts) (width 0.1))
+  (gr_arc (start 166 22.25) (end 166 17.25) (angle 90) (layer Edge.Cuts) (width 0.1))
   (gr_line (start 260 98.25) (end 265 93.25) (angle 90) (layer Edge.Cuts) (width 0.1))
   (gr_line (start 265 93.25) (end 329.25 93.25) (angle 90) (layer Edge.Cuts) (width 0.1))
@@
   (gr_line (start 215.5 125.5) (end 220.5 120.5) (angle 90) (layer Edge.Cuts) (width 0.1))
   (gr_line (start 215.5 125.5) (end 185.5 125.5) (angle 90) (layer Edge.Cuts) (width 0.1))
-  (gr_line (start 180.25 120.5) (end 185.25 125.5) (angle 90) (layer Edge.Cuts) (width 0.1))
   (gr_line (start 185.25 125.5) (end 185.5 125.5) (angle 90) (layer Edge.Cuts) (width 0.1))
   (gr_line (start 180.25 120.5) (end 180.25 22.25) (angle 90) (layer Edge.Cuts) (width 0.1))
-  (gr_line (start 180.25 22.25) (end 185.25 17.25) (angle 90) (layer Edge.Cuts) (width 0.1))
   (gr_line (start 185.25 17.25) (end 225.75 17.25) (angle 90) (layer Edge.Cuts) (width 0.1))
   (gr_line (start 225.75 17.25) (end 231 12) (angle 90) (layer Edge.Cuts) (width 0.1))
@@
   (gr_line (start 302.25 19.75) (end 334 19.75) (angle 90) (layer Edge.Cuts) (width 0.1))
   (gr_line (start 339 24.75) (end 339 88.5) (angle 90) (layer Edge.Cuts) (width 0.1))
-  (gr_line (start 339 88.5) (end 334.25 93.25) (angle 90) (layer Edge.Cuts) (width 0.1))
   (gr_line (start 334.25 93.25) (end 329.25 93.25) (angle 90) (layer Edge.Cuts) (width 0.1))
-  (gr_line (start 339 24.75) (end 334 19.75) (angle 90) (layer Edge.Cuts) (width 0.1))
-  (gr_line (start 12.25 24.75) (end 17.25 19.75) (angle 90) (layer Edge.Cuts) (width 0.1))
   (gr_line (start 17 93.25) (end 22 93.25) (angle 90) (layer Edge.Cuts) (width 0.1))
-  (gr_line (start 12.25 88.5) (end 17 93.25) (angle 90) (layer Edge.Cuts) (width 0.1))
   (gr_line (start 12.25 24.75) (end 12.25 88.5) (angle 90) (layer Edge.Cuts) (width 0.1))
   (gr_line (start 49 19.75) (end 17.25 19.75) (angle 90) (layer Edge.Cuts) (width 0.1))
@@
   (gr_line (start 125.5 17.25) (end 120.25 12) (angle 90) (layer Edge.Cuts) (width 0.1))
   (gr_line (start 166 17.25) (end 125.5 17.25) (angle 90) (layer Edge.Cuts) (width 0.1))
-  (gr_line (start 171 22.25) (end 166 17.25) (angle 90) (layer Edge.Cuts) (width 0.1))
   (gr_line (start 171 120.5) (end 171 22.25) (angle 90) (layer Edge.Cuts) (width 0.1))
   (gr_line (start 166 125.5) (end 165.75 125.5) (angle 90) (layer Edge.Cuts) (width 0.1))
-  (gr_line (start 171 120.5) (end 166 125.5) (angle 90) (layer Edge.Cuts) (width 0.1))
   (gr_line (start 135.75 125.5) (end 165.75 125.5) (angle 90) (layer Edge.Cuts) (width 0.1))
   (gr_line (start 135.75 125.5) (end 130.75 120.5) (angle 90) (layer Edge.Cuts) (width 0.1))
@@
   (segment (start 203.75 100) (end 194.5 100) (width 0.25) (layer B.Cu) (net 89))
   (segment (start 204.77 101.02) (end 203.75 100) (width 0.25) (layer B.Cu) (net 89))
-  (segment (start 146.75 29.5) (end 146.75 33) (width 0.25) (layer F.Cu) (net 97))
   (segment (start 149.3 24.96) (end 149.3 26.22) (width 0.25) (layer F.Cu) (net 97))
   (segment (start 149.3 26.22) (end 149.25 26.27) (width 0.25) (layer F.Cu) (net 97))
@@
   (segment (start 153 28.25) (end 154 28.25) (width 0.25) (layer F.Cu) (net 97))
   (segment (start 151.75 27) (end 153 28.25) (width 0.25) (layer F.Cu) (net 97))
+  (segment (start 161.25 30.75) (end 161.25 33) (width 0.25) (layer F.Cu) (net 97))
+  (segment (start 160.25 29.75) (end 161.25 30.75) (width 0.25) (layer F.Cu) (net 97))
+  (segment (start 158.25 29.75) (end 160.25 29.75) (width 0.25) (layer F.Cu) (net 97))
+  (segment (start 156.75 28.25) (end 158.25 29.75) (width 0.25) (layer F.Cu) (net 97))
+  (segment (start 154 28.25) (end 156.75 28.25) (width 0.25) (layer F.Cu) (net 97))
+  (segment (start 146.75 29.5) (end 146.75 33) (width 0.25) (layer F.Cu) (net 98))
   (segment (start 147.7 24.96) (end 147.7 26.22) (width 0.25) (layer F.Cu) (net 98))
   (segment (start 147.7 26.22) (end 147.75 26.27) (width 0.25) (layer F.Cu) (net 98))
@@
   (segment (start 147.75 28) (end 147.75 28.5) (width 0.25) (layer F.Cu) (net 98))
   (segment (start 147.75 28.5) (end 146.75 29.5) (width 0.25) (layer F.Cu) (net 98))
-  (segment (start 161.25 30.75) (end 161.25 33) (width 0.25) (layer F.Cu) (net 98))
-  (segment (start 160.25 29.75) (end 161.25 30.75) (width 0.25) (layer F.Cu) (net 98))
-  (segment (start 158.25 29.75) (end 160.25 29.75) (width 0.25) (layer F.Cu) (net 98))
-  (segment (start 156.75 28.25) (end 158.25 29.75) (width 0.25) (layer F.Cu) (net 98))
-  (segment (start 154 28.25) (end 156.75 28.25) (width 0.25) (layer F.Cu) (net 98))
   (segment (start 150.1 24.96) (end 150.1 25.1) (width 0.25) (layer F.Cu) (net 99))
   (segment (start 150.1 25.1) (end 150.75 25.75) (width 0.25) (layer F.Cu) (net 99))

Commit message: moved receptacles to the back side, rewired connections
Parts:
- J1, J2, J3: moved to B.Cu
- moved J1 1.75 mm to (150.5, 23.0), turned to 0 degrees
- moved J2 1.75 mm to (165.2, 90.0), turned to 270 degrees
- moved J3 1.75 mm to (186.0, 90.0), turned to 90 degrees
Connections:
- J2 pad A2: /row1 -> /row0
- J2 pad A3: /row0 -> /row1
- J2 pad A4: /col6 -> Net-(J2-PadA4)
- J2 pad A5: /col7 -> Net-(J2-PadA5)
- J2 pad A6: /col8 -> Net-(J2-PadA6)
- J2 pad A7: /col9 -> Net-(J2-PadA7)
- J2 pad A8: /colA -> Net-(J2-PadA8)
- J2 pad A9: /colB -> Net-(J2-PadA9)
- J2 pad B10: /row2 -> /colA
- J2 pad B11: /row3 -> /colB
- J2 pad B2: /row1 -> /col6
- J2 pad B3: /row0 -> /col7
- J2 pad B4: /col6 -> Net-(J2-PadB4)
- J2 pad B5: /col7 -> Net-(J2-PadB5)
- J2 pad B8: /colA -> Net-(J2-PadB8)
- J2 pad B9: /colB -> Net-(J2-PadB9)
- J3 pad A10: /row2 -> /col7
- J3 pad A11: /row3 -> /col6
- J3 pad A2: /row1 -> /colB
- J3 pad A3: /row0 -> /colA
- J3 pad A4: /col6 -> Net-(J3-PadA4)
- J3 pad A5: /col7 -> Net-(J3-PadA5)
- J3 pad A6: /col8 -> Net-(J3-PadA6)
- J3 pad A7: /col9 -> Net-(J3-PadA7)
- J3 pad A8: /colA -> Net-(J3-PadA8)
- J3 pad A9: /colB -> Net-(J3-PadA9)
- J3 pad B10: /row2 -> /row1
- J3 pad B11: /row3 -> /row0
- J3 pad B2: /row1 -> /row3
- J3 pad B3: /row0 -> /row2
- J3 pad B4: /col6 -> Net-(J3-PadB4)
- J3 pad B5: /col7 -> Net-(J3-PadB5)
- J3 pad B8: /colA -> Net-(J3-PadB8)
- J3 pad B9: /colB -> Net-(J3-PadB9)
Routing:
- net /colB: track 357.5 -> 231.0 mm, vias 7 -> 3
- net /col7: track 278.1 -> 157.4 mm, vias 5 -> 3
- net /colA: track 332.2 -> 214.3 mm, vias 7 -> 3
- net /col9: track 302.8 -> 222.6 mm, vias 7 -> 4
- net /row2: track 427.5 -> 354.4 mm, vias 9 -> 5
- net /col8: track 315.1 -> 249.1 mm, vias 7 -> 4
- net /col6: track 220.2 -> 157.3 mm, vias 5 -> 1
- net /row0: track 500.6 -> 437.8 mm, vias 5 -> 2
- net /row1: track 444.3 -> 387.4 mm
- net /row3: track 255.5 -> 207.8 mm, vias 2 -> 0
- net /D-: track 20.1 -> 14.0 mm, vias 2 -> 1
- net /+5v: track 24.0 -> 27.4 mm
- net /D+: track 8.62 -> 7.08 mm
- net Net-(D42-Pad2): track 17.6 -> 18.9 mm
- net /GND: track 16.4 -> 17.3 mm, vias 2 -> 0
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Other:
- board text added: "github.com/nglgzz/42"
