File: pcb/kicad/pcb.kicad_pcb (KiCad board)
At the start: 2 copper layers, 303 x 103 mm, 85 parts, among them K0 KEYSW, K0A1 KEYSW, K0B1 KEYSW, K1 KEYSW, K10 KEYSW, K11 KEYSW, K12 KEYSW, K13 KEYSW, K14 KEYSW, K15 KEYSW, K16 KEYSW, K17 KEYSW, K18 KEYSW, K19 KEYSW, K1A1 KEYSW, K1B1 KEYSW, K2 KEYSW, K20 KEYSW, K21 KEYSW, K22 KEYSW, K23 KEYSW, K24 KEYSW, K25 KEYSW, K26 KEYSW, K27 KEYSW, K28 KEYSW, K29 KEYSW, K2A1 KEYSW, K2B1 KEYSW, K3 KEYSW, K33 KEYSW, K34 KEYSW, K35 KEYSW, K36 KEYSW, K37 KEYSW, K38 KEYSW, K4 KEYSW, K5 KEYSW, K6 KEYSW, K7 KEYSW, K8 KEYSW, K9 KEYSW, U1 Feather_32u4_BLE

Commit message: Redesign PCB for Elite-C
Parts:
- U1: value Feather_32u4_BLE -> Elite-C; footprint pcb:Feather_32u4_BLE -> Keebio-Parts:Elite-C-castellated-29pin-holes
- moved U1 7.12 mm to (161.0, 79.5), turned to 270 degrees
Connections:
- U1 pad 10: Net-(U1-Pad10) -> /col3
- U1 pad 11: Net-(U1-Pad11) -> /col4
- U1 pad 12: Net-(U1-Pad12) -> /col5
- U1 pad 13: /row0 -> /col6
- U1 pad 14: /row1 -> /col7
- U1 pad 15: Net-(U1-Pad15) -> /col8
- U1 pad 16: Net-(U1-Pad16) -> /col9
- U1 pad 17: Net-(U1-Pad17) -> /colA
- U1 pad 18: Net-(U1-Pad18) -> /colB
- U1 pad 19: /col9 -> Net-(U1-Pad19)
- U1 pad 20: /colA -> Net-(U1-Pad20)
- U1 pad 21: /colB -> Net-(U1-Pad21)
- U1 pad 22: /col6 -> Net-(U1-Pad22)
- U1 pad 23: /col7 -> Net-(U1-Pad23)
- U1 pad 24: /col8 -> Net-(U1-Pad24)
- U1 pad 25: Net-(U1-Pad25) -> /row0
- U1 pad 26: /row2 -> Net-(U1-Pad26)
- U1 pad 27: /row3 -> /row1
- U1 pad 4: /col2 -> Net-(U1-Pad4)
- U1 pad 5: /col1 -> Net-(U1-Pad5)
- U1 pad 6: /col0 -> Net-(U1-Pad6)
- U1 pad 7: /col5 -> /col0
- U1 pad 8: /col4 -> /col1
- U1 pad 9: /col3 -> /col2
Routing:
- net /row0: track 365.8 -> 472.1 mm, vias 0 -> 4
- net /row3: track 207.9 -> 266.8 mm, vias 0 -> 1
- net /row1: track 373.1 -> 430.1 mm, vias 6 -> 5
- net /row2: track 480.4 -> 534.0 mm
- net /col2: track 164.7 -> 147.2 mm, vias 3 -> 1
- net /col4: track 156.5 -> 142.8 mm, vias 3 -> 1
- net /col0: track 184.9 -> 194.5 mm, vias 3 -> 1
- net /col9: track 148.0 -> 139.6 mm, vias 3 -> 1
- net /col7: track 140.5 -> 133.6 mm, vias 3 -> 1
- net /col5: track 127.6 -> 133.5 mm, vias 3 -> 1
- net /col8: track 148.9 -> 154.7 mm
- net /colB: track 182.1 -> 177.5 mm
- net /col1: track 162.7 -> 167.3 mm, vias 3 -> 1
- net /col3: track 168.1 -> 163.8 mm, vias 3 -> 1
- net Net-(U1-Pad26): track 0.00 -> 1.91 mm
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Other:
- outline, holes or cut-outs redrawn
- board text added: "nglgzz 42 v3.2"
- board text removed: "nglgzz 42"

Commit message: Add support for Choc v1 switches
Parts:
- K0, K0A1, K0B1, K1, K10, K11, K12, K13, K14, K15, K16, K17, K18, K19, K1A1, K1B1, K2, K20, K21, K22, K23, K24, K25, K26, K27, K28, K29, K2A1, K2B1, K3, K33, K34, K35, K36, K37, K38, K4, K5, K6, K7, K8, K9: footprint Keebs:Mx_Alps_100 -> Keebio-Parts:MX-Alps-Choc-1U-NoLED
Routing:
- net /col6: track 126.5 -> 143.5 mm
- net /col4: track 142.8 -> 159.8 mm
- net /col3: track 163.8 -> 180.8 mm
- net /col5: track 133.5 -> 150.5 mm
- net /col7: track 133.6 -> 150.0 mm
- net Net-(D9-Pad2): track 12.4 -> 27.2 mm
- net /colB: track 177.5 -> 190.2 mm
- net /colA: track 160.0 -> 172.8 mm
- net /col9: track 139.6 -> 152.3 mm
- net /col2: track 147.2 -> 159.9 mm
- net /col1: track 167.3 -> 180.0 mm
- net /col0: track 194.5 -> 207.3 mm
- net /col8: track 154.7 -> 167.2 mm
- net Net-(D26-Pad2): track 14.1 -> 18.6 mm
- net Net-(D1B1-Pad2): track 13.7 -> 17.7 mm
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
Commit message: Add PCB support for Pro Micro
Connections:
- U1 pad 10: /col3 -> /col5
- U1 pad 11: /col4 -> /row0
- U1 pad 12: /col5 -> /row1
- U1 pad 13: /col6 -> /row3
- U1 pad 14: /col7 -> /row2
- U1 pad 15: /col8 -> /col6
- U1 pad 16: /col9 -> /col7
- U1 pad 17: /colA -> /col8
- U1 pad 18: /colB -> /col9
- U1 pad 19: Net-(U1-Pad19) -> /colA
- U1 pad 20: Net-(U1-Pad20) -> /colB
- U1 pad 25: /row0 -> Net-(U1-Pad25)
- U1 pad 27: /row1 -> Net-(U1-Pad27)
- U1 pad 28: /row2 -> Net-(U1-Pad28)
- U1 pad 29: /row3 -> Net-(U1-Pad29)
- U1 pad 5: Net-(U1-Pad5) -> /col0
- U1 pad 6: Net-(U1-Pad6) -> /col1
- U1 pad 7: /col0 -> /col2
- U1 pad 8: /col1 -> /col3
- U1 pad 9: /col2 -> /col4
Routing:
- net /row2: track 534.0 -> 522.6 mm
- net /row3: track 266.8 -> 256.4 mm
- net /col0: track 207.3 -> 200.1 mm
- net /row1: track 430.1 -> 423.8 mm
- net Net-(U1-Pad27): track 0.00 -> 2.19 mm
- net Net-(U1-Pad29): track 0.00 -> 2.14 mm
- net /row0: track 472.1 -> 470.0 mm
- net /col9: track 152.3 -> 150.2 mm
- net /col8: track 167.2 -> 169.3 mm
- net /col7: track 150.0 -> 152.1 mm
- net /col2: track 159.9 -> 157.8 mm
- net /col4: track 159.8 -> 161.9 mm
- net /col3: track 180.8 -> 182.9 mm
- net Net-(U1-Pad28): track 0.00 -> 1.91 mm
- net Net-(U1-Pad25): track 0.00 -> 1.91 mm
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
Commit message: Update gerber files
Other:
- outline, holes or cut-outs redrawn
- board text added: "nglgzz/42 v3.1"
- board text removed: "nglgzz 42 v3.2"
